File: PCB/Motor relay/standalone.brd (EAGLE design)
At the start: 160 x 100 mm, 11 parts, among them J1 1X2-3.5MM, U1 328P, Y1 16MHz

Commit message: MOD2
Parts:
- added LED1, LED3: (no value), adafruit:LED5MM
- added R2: (no value), resistor:0204/5
- added R3: (no value), adafruit:0204/7
Connections:
- new net N$1: LED3.A, R3.2
- new net N$3: R2.1, U1.23
- new net N$4: LED1.A, R2.2
- new net N$5: R3.1, U1.24
- net GND: now also LED1.K, LED3.K
Changed lines of the file:
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@@
 <attribute name="OC_NEWARK" value="97K7059" x="-5.08" y="7.62" size="1.778" layer="27" display="off"/>
 </element>
+<element name="R2" library="resistor" library_urn="urn:adsk.eagle:library:348" package="0204/5" package3d_urn="urn:adsk.eagle:package:25955/1" value="" x="-5.08" y="-3.81"/>
+<element name="LED3" library="adafruit" library_urn="urn:adsk.eagle:library:420" package="LED5MM" value="" x="-6.35" y="-24.13"/>
+<element name="R3" library="adafruit" library_urn="urn:adsk.eagle:library:420" package="0204/7" value="" x="-3.81" y="-30.48"/>
+<element name="LED1" library="adafruit" library_urn="urn:adsk.eagle:library:420" package="LED5MM" value="" x="-6.35" y="-35.56"/>
 </elements>
 <signals>
@@
 <contactref element="OK1" pad="2"/>
 <contactref element="JP1" pad="2"/>
+<contactref element="LED3" pad="K"/>
+<contactref element="LED1" pad="K"/>
 <wire x1="35.56" y1="20.32" x2="48.26" y2="29.36875" width="0" layer="19" extent="16-16"/>
 <wire x1="-3.81" y1="3.81" x2="35.56" y2="20.32" width="0" layer="19" extent="1-1"/>
+<wire x1="-5.08" y1="-24.13" x2="-3.81" y2="3.81" width="0" layer="19" extent="1-1"/>
+<wire x1="-5.08" y1="-35.56" x2="-5.08" y2="-24.13" width="0" layer="19" extent="1-1"/>
 </signal>
 <signal name="VCC">
@@
 <wire x1="-3.81" y1="11.43" x2="33.02" y2="20.32" width="0" layer="19" extent="1-1"/>
 </signal>
+<signal name="N$3">
+<contactref element="U1" pad="23"/>
+<contactref element="R2" pad="1"/>
+<wire x1="-7.62" y1="-3.81" x2="50.8" y2="44.45" width="0" layer="19" extent="1-1"/>
+</signal>
+<signal name="N$4">
+<contactref element="R2" pad="2"/>
+<contactref element="LED1" pad="A"/>
+<wire x1="-2.54" y1="-3.81" x2="-7.62" y2="-35.56" width="0" layer="19" extent="1-1"/>
+</signal>
+<signal name="N$1">
+<contactref element="R3" pad="2"/>
+<contactref element="LED3" pad="A"/>
+<wire x1="-7.62" y1="-24.13" x2="0" y2="-30.48" width="0" layer="19" extent="1-1"/>
+</signal>
+<signal name="N$5">
+<contactref element="R3" pad="1"/>
+<contactref element="U1" pad="24"/>
+<wire x1="-7.62" y1="-30.48" x2="48.26" y2="44.45" width="0" layer="19" extent="1-1"/>
+</signal>
 </signals>
