File: PCB/Motor relay/standalone.sch (EAGLE design)
At the start: 12 parts, among them J1 1X2-3.5MM, U1 328P, Y1 16MHz

Commit message: PCB MOD1
Parts:
- removed C4: 1uF, SparkFun-Capacitors:10UF-POLAR-RADIAL-2.5MM-25V-20%
- removed U2: (no value), SparkFun-IC-Power:V_REG_78XXSINK
- added OK1: PC817, optocoupler:PC817
Connections:
- removed net RELAY: JP1.2, U1.PD3(INT1)
- new net RELAYSIG: OK1.A, U1.PD3(INT1)
- net GND: now also JP1.2, OK1.C; no longer C4.+, JP1.3, U2.GND
- net N$2: now also JP1.1, OK1.EMIT; no longer C4.-, J1.2, U2.IN
- net VCC: now also J1.2, OK1.COL; no longer JP1.1, U2.OUT
Other:
- note removed: "Power supply"
- moved on the sheet: JP1
Changed lines of the file:
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@@
 <part name="C2" library="SparkFun-Capacitors" library_urn="urn:adsk.eagle:library:510" deviceset="22PF" device="-PTH-2.54MM-200V-5%" package3d_urn="urn:adsk.eagle:package:37435/1" value="22pF"/>
 <part name="SUPPLY1" library="supply2" library_urn="urn:adsk.eagle:library:372" deviceset="GND" device=""/>
-<part name="U2" library="SparkFun-IC-Power" library_urn="urn:adsk.eagle:library:526" deviceset="V_REG_78XX" device="SINK" package3d_urn="urn:adsk.eagle:package:39063/1"/>
 <part name="J1" library="adafruit" library_urn="urn:adsk.eagle:library:420" deviceset="1X2" device="-3.5MM"/>
 <part name="P+1" library="supply1" library_urn="urn:adsk.eagle:library:371" deviceset="VCC" device=""/>
@@
 <part name="S1" library="switch-omron" library_urn="urn:adsk.eagle:library:377" deviceset="10-XX" device="" package3d_urn="urn:adsk.eagle:package:27496/1"/>
 <part name="C3" library="SparkFun-Capacitors" library_urn="urn:adsk.eagle:library:510" deviceset="10UF-POLAR" device="-RADIAL-2.5MM-25V-20%" package3d_urn="urn:adsk.eagle:package:37423/1" value="10uF"/>
-<part name="C4" library="SparkFun-Capacitors" library_urn="urn:adsk.eagle:library:510" deviceset="10UF-POLAR" device="-RADIAL-2.5MM-25V-20%" package3d_urn="urn:adsk.eagle:package:37423/1" value="1uF"/>
 <part name="JP1" library="adafruit" library_urn="urn:adsk.eagle:library:420" deviceset="PINHD-1X3" device=""/>
+<part name="OK1" library="optocoupler" library_urn="urn:adsk.eagle:library:320" deviceset="PC817" device="" package3d_urn="urn:adsk.eagle:package:21938/1"/>
+<part name="SUPPLY4" library="supply2" library_urn="urn:adsk.eagle:library:372" deviceset="GND" device=""/>
+<part name="SUPPLY5" library="supply2" library_urn="urn:adsk.eagle:library:372" deviceset="GND" device=""/>
 </parts>
 <sheets>
@@
 <plain>
 <text x="27.94" y="91.44" size="1.778" layer="91">Clock</text>
-<text x="25.4" y="127" size="1.778" layer="91">Power supply</text>
 <text x="58.42" y="127" size="1.778" layer="91">RESET</text>
 <text x="55.88" y="93.98" size="1.778" layer="91">Programming headers</text>
@@
 <instance part="C2" gate="G$1" x="25.4" y="73.66"/>
 <instance part="SUPPLY1" gate="GND" x="30.48" y="63.5"/>
-<instance part="U2" gate="G$1" x="33.02" y="121.92"/>
 <instance part="J1" gate="G$1" x="30.48" y="104.14" rot="R270"/>
 <instance part="P+1" gate="VCC" x="45.72" y="124.46"/>
@@
 <instance part="S1" gate="1" x="73.66" y="104.14" rot="R90"/>
 <instance part="C3" gate="G$1" x="43.18" y="116.84" rot="R180"/>
-<instance part="C4" gate="G$1" x="30.48" y="111.76" rot="R270"/>
-<instance part="JP1" gate="A" x="99.06" y="66.04"/>
+<instance part="JP1" gate="A" x="127" y="40.64"/>
+<instance part="OK1" gate="A" x="91.44" y="43.18"/>
+<instance part="SUPPLY4" gate="GND" x="76.2" y="30.48"/>
+<instance part="SUPPLY5" gate="GND" x="121.92" y="27.94"/>
 </instances>
 <busses>
@@
 </segment>
 <segment>
-<pinref part="U2" gate="G$1" pin="GND"/>
-<pinref part="J1" gate="G$1" pin="1"/>
-<wire x1="33.02" y1="114.3" x2="33.02" y2="111.76" width="0.1524" layer="91"/>
-<wire x1="33.02" y1="111.76" x2="33.02" y2="109.22" width="0.1524" layer="91"/>
-<junction x="33.02" y="111.76"/>
 <wire x1="43.18" y1="114.3" x2="43.18" y2="111.76" width="0.1524" layer="91"/>
 <pinref part="SUPPLY2" gate="GND" pin="GND"/>
-<wire x1="43.18" y1="111.76" x2="33.02" y2="111.76" width="0.1524" layer="91"/>
-<junction x="43.18" y="111.76"/>
 <pinref part="C3" gate="G$1" pin="+"/>
-<pinref part="C4" gate="G$1" pin="+"/>
+<pinref part="J1" gate="G$1" pin="1"/>
+<wire x1="33.02" y1="109.22" x2="33.02" y2="111.76" width="0.1524" layer="91"/>
+<wire x1="33.02" y1="111.76" x2="43.18" y2="111.76" width="0.1524" layer="91"/>
 </segment>
 <segment>
@@
 </segment>
 <segment>
-<pinref part="JP1" gate="A" pin="3"/>
-<wire x1="96.52" y1="63.5" x2="88.9" y2="63.5" width="0.1524" layer="91"/>
-<label x="88.9" y="63.5" size="1.778" layer="95" rot="R180" xref="yes"/>
-</segment>
-</net>
-<net name="N$2" class="0">
-<segment>
-<pinref part="J1" gate="G$1" pin="2"/>
-<pinref part="U2" gate="G$1" pin="IN"/>
-<wire x1="25.4" y1="121.92" x2="20.32" y2="121.92" width="0.1524" layer="91"/>
-<wire x1="20.32" y1="121.92" x2="20.32" y2="111.76" width="0.1524" layer="91"/>
-<wire x1="20.32" y1="111.76" x2="20.32" y2="109.22" width="0.1524" layer="91"/>
-<wire x1="20.32" y1="109.22" x2="30.48" y2="109.22" width="0.1524" layer="91"/>
-<wire x1="25.4" y1="111.76" x2="20.32" y2="111.76" width="0.1524" layer="91"/>
-<pinref part="C4" gate="G$1" pin="-"/>
+<pinref part="OK1" gate="A" pin="C"/>
+<wire x1="81.28" y1="40.64" x2="76.2" y2="40.64" width="0.1524" layer="91"/>
+<wire x1="76.2" y1="40.64" x2="76.2" y2="33.02" width="0.1524" layer="91"/>
+<pinref part="SUPPLY4" gate="GND" pin="GND"/>
+</segment>
+<segment>
+<pinref part="JP1" gate="A" pin="2"/>
+<wire x1="124.46" y1="40.64" x2="121.92" y2="40.64" width="0.1524" layer="91"/>
+<wire x1="121.92" y1="40.64" x2="121.92" y2="30.48" width="0.1524" layer="91"/>
+<pinref part="SUPPLY5" gate="GND" pin="GND"/>
 </segment>
 </net>
 <net name="VCC" class="0">
 <segment>
-<pinref part="U2" gate="G$1" pin="OUT"/>
 <pinref part="P+1" gate="VCC" pin="VCC"/>
-<wire x1="40.64" y1="121.92" x2="43.18" y2="121.92" width="0.1524" layer="91"/>
 <pinref part="C3" gate="G$1" pin="-"/>
 <wire x1="43.18" y1="121.92" x2="45.72" y2="121.92" width="0.1524" layer="91"/>
 <junction x="43.18" y="121.92"/>
+<pinref part="J1" gate="G$1" pin="2"/>
+<wire x1="30.48" y1="109.22" x2="30.48" y2="121.92" width="0.1524" layer="91"/>
+<wire x1="30.48" y1="121.92" x2="43.18" y2="121.92" width="0.1524" layer="91"/>
 </segment>
 <segment>
@@
 </segment>
 <segment>
-<pinref part="JP1" gate="A" pin="1"/>
-<wire x1="96.52" y1="68.58" x2="88.9" y2="68.58" width="0.1524" layer="91"/>
-<label x="88.9" y="68.58" size="1.778" layer="95" rot="R180" xref="yes"/>
+<pinref part="OK1" gate="A" pin="COL"/>
+<wire x1="99.06" y1="45.72" x2="104.14" y2="45.72" width="0.1524" layer="91"/>
+<label x="104.14" y="45.72" size="1.778" layer="95" xref="yes"/>
+<label x="104.14" y="45.72" size="1.778" layer="95" xref="yes"/>
+<label x="104.14" y="45.72" size="1.778" layer="95" xref="yes"/>
+<label x="104.14" y="45.72" size="1.778" layer="95" xref="yes"/>
 </segment>
 </net>
@@
 </segment>
 </net>
-<net name="RELAY" class="0">
+<net name="RELAYSIG" class="0">
 <segment>
 <pinref part="U1" gate="G$1" pin="PD3(INT1)"/>
@@
 </segment>
 <segment>
-<pinref part="JP1" gate="A" pin="2"/>
-<wire x1="96.52" y1="66.04" x2="88.9" y2="66.04" width="0.1524" layer="91"/>
-<label x="88.9" y="66.04" size="1.778" layer="95" rot="R180" xref="yes"/>
-</segment>
-</net>
+<pinref part="OK1" gate="A" pin="A"/>
+<wire x1="81.28" y1="45.72" x2="76.2" y2="45.72" width="0.1524" layer="91"/>
+<label x="76.2" y="45.72" size="1.778" layer="95" rot="R180" xref="yes"/>
+</segment>
+</net>
+<net name="N$2" class="0">
+<segment>
+<pinref part="OK1" gate="A" pin="EMIT"/>
+<wire x1="99.06" y1="40.64" x2="119.38" y2="40.64" width="0.1524" layer="91"/>
+<wire x1="119.38" y1="40.64" x2="119.38" y2="43.18" width="0.1524" layer="91"/>
+<pinref part="JP1" gate="A" pin="1"/>
+<wire x1="124.46" y1="43.18" x2="119.38" y2="43.18" width="0.1524" layer="91"/>
+</segment>
+</net>

Commit message: MOD2
Parts:
- added LED1, LED3: (no value), adafruit:LED5MM
- added R2: (no value), resistor:R-US_0204/5
- added R3: (no value), adafruit:R-US_0204/7
Connections:
- new net N$1: LED3.A, R3.2
- new net N$3: R2.1, U1.PC0(ADC0)
- new net N$4: LED1.A, R2.2
- new net N$5: R3.1, U1.PC1(ADC1)
- net GND: now also LED1.C, LED3.C
Changed lines of the file:
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@@
 <part name="SUPPLY4" library="supply2" library_urn="urn:adsk.eagle:library:372" deviceset="GND" device=""/>
 <part name="SUPPLY5" library="supply2" library_urn="urn:adsk.eagle:library:372" deviceset="GND" device=""/>
+<part name="R2" library="resistor" library_urn="urn:adsk.eagle:library:348" deviceset="R-US_" device="0204/5" package3d_urn="urn:adsk.eagle:package:25955/1"/>
+<part name="SUPPLY6" library="supply2" library_urn="urn:adsk.eagle:library:372" deviceset="GND" device=""/>
+<part name="SUPPLY7" library="supply2" library_urn="urn:adsk.eagle:library:372" deviceset="GND" device=""/>
+<part name="LED3" library="adafruit" library_urn="urn:adsk.eagle:library:420" deviceset="LED" device="5MM"/>
+<part name="R3" library="adafruit" library_urn="urn:adsk.eagle:library:420" deviceset="R-US_" device="0204/7"/>
+<part name="LED1" library="adafruit" library_urn="urn:adsk.eagle:library:420" deviceset="LED" device="5MM"/>
 </parts>
 <sheets>
@@
 <instance part="SUPPLY4" gate="GND" x="76.2" y="30.48"/>
 <instance part="SUPPLY5" gate="GND" x="121.92" y="27.94"/>
+<instance part="R2" gate="G$1" x="182.88" y="127"/>
+<instance part="SUPPLY6" gate="GND" x="193.04" y="114.3"/>
+<instance part="SUPPLY7" gate="GND" x="185.42" y="109.22"/>
+<instance part="LED3" gate="G$1" x="185.42" y="119.38"/>
+<instance part="R3" gate="G$1" x="180.34" y="124.46"/>
+<instance part="LED1" gate="G$1" x="193.04" y="124.46"/>
 </instances>
 <busses>
@@
 <pinref part="SUPPLY5" gate="GND" pin="GND"/>
 </segment>
+<segment>
+<pinref part="SUPPLY6" gate="GND" pin="GND"/>
+<wire x1="193.04" y1="119.38" x2="193.04" y2="116.84" width="0.1524" layer="91"/>
+<pinref part="LED1" gate="G$1" pin="C"/>
+</segment>
+<segment>
+<pinref part="LED3" gate="G$1" pin="C"/>
+<pinref part="SUPPLY7" gate="GND" pin="GND"/>
+<wire x1="185.42" y1="114.3" x2="185.42" y2="111.76" width="0.1524" layer="91"/>
+</segment>
 </net>
 <net name="VCC" class="0">
@@
 </segment>
 </net>
+<net name="N$3" class="0">
+<segment>
+<pinref part="U1" gate="G$1" pin="PC0(ADC0)"/>
+<wire x1="172.72" y1="127" x2="177.8" y2="127" width="0.1524" layer="91"/>
+<pinref part="R2" gate="G$1" pin="1"/>
+</segment>
+</net>
+<net name="N$4" class="0">
+<segment>
+<pinref part="R2" gate="G$1" pin="2"/>
+<wire x1="193.04" y1="127" x2="187.96" y2="127" width="0.1524" layer="91"/>
+<pinref part="LED1" gate="G$1" pin="A"/>
+</segment>
+</net>
+<net name="N$1" class="0">
+<segment>
+<pinref part="R3" gate="G$1" pin="2"/>
+<pinref part="LED3" gate="G$1" pin="A"/>
+<wire x1="185.42" y1="124.46" x2="185.42" y2="121.92" width="0.1524" layer="91"/>
+</segment>
+</net>
+<net name="N$5" class="0">
+<segment>
+<pinref part="R3" gate="G$1" pin="1"/>
+<pinref part="U1" gate="G$1" pin="PC1(ADC1)"/>
+<wire x1="175.26" y1="124.46" x2="172.72" y2="124.46" width="0.1524" layer="91"/>
+</segment>
+</net>
